Commit message: added Intel RealSense D455 camera in right_arm.urdf.xacro and added new camera pose

File: turbo_description/urdf/right_arm.urdf.xacro (robot description, xacro)
@@ -35,4 +35,9 @@
   <!-- robotiq 85 -->
   <xacro:include filename="$(find robotiq_85_description)/urdf/robotiq_85_gripper.urdf.xacro"/>
+  <!-- Intel RealSense D455 camera -->
+  <xacro:include filename="$(find realsense2_description)/urdf/_d455.urdf.xacro"/>
+  <xacro:sensor_d455 parent="camera_mount">
+    <origin xyz="0 0 0" rpy="0 0 0"/>
+  </xacro:sensor_d455>
   <link name="world"/>
   <link name="frame">
@@ -97,10 +102,10 @@
     <origin xyz="0.265 0.635 1.275" rpy="-0.785 3.14 1.57"/>
   </joint>
-  <!-- astra camera -->
+  <!-- Intel RealSense D455 camera -->
   <link name="camera_mount"/>
   <joint name="camera_to_frame" type="fixed">
     <parent link="frame"/>
     <child link = "camera_mount"/>
-    <origin xyz="0.54 0.54 1.45" rpy="0 1.30 -1.57"/>
+    <origin xyz="0.47 -0.11 1.195" rpy="0 ${47.5*pi/180} ${90*pi/180}"/>
   </joint>
   <link name="right_ee_link"/>
@@ -113,6 +118,3 @@
     <origin xyz="0 0 0" rpy="0 0 0"/>
   </xacro:robotiq_85_gripper>
-  <!-- Astra camera -->
-  <xacro:include filename="$(find turbo_description)/urdf/camera/astra.xacro"/>
-  <xacro:sensor_astra name="astra" parent="camera_mount" cam_px="0.01" cam_pz="${0.052}" meshes="package://turbo_description/meshes/rgbd" />
 </robot>
